Commit message: Fixed multi mir spawn by using fork of robot_state_publisher https://github.com/ros/robot_state_publisher/pull/139

File: mir/mir_description/urdf/general/sick_s300.gazebo.xacro (robot description, xacro)
@@ -2,5 +2,5 @@
 <robot xmlns:xacro="http://ros.org/wiki/xacro">
 	<xacro:include filename="$(find mir_description)/urdf/general/common_properties.urdf.xacro" />
-	<xacro:macro name="sick_s300_gazebo" params="link topic robot_namespace">
+	<xacro:macro name="sick_s300_gazebo" params="link topic robot_namespace tf_prefix">
 		<gazebo reference="${link}">
 			<xacro:insert_block name="material_black" />
@@ -35,5 +35,5 @@
 					<!-- no tf_prefix, plugin always uses a tf_prefix (if none is set it uses robotNamespace) -->
 					<robotNamespace>${robot_namespace}</robotNamespace>
-					<frameName>${link}</frameName>
+					<frameName>${tf_prefix}/${link}</frameName>
 					<topicName>${topic}</topicName>
 				</plugin>

File: mir/mir_description/urdf/mir_100/mir_100.gazebo.xacro (robot description, xacro)
@@ -44,6 +44,6 @@
 		<!-- Add Gazebo xacro for the laser scanner to work in Gazebo -->
 		<!-- Please match there macro calls with the sick_s300 xacro calls in the mir_100.urdf.xacro file-->
-		<xacro:sick_s300_gazebo link="front_laser_link" robot_namespace="${robot_namespace_slashed}" topic="f_scan" />
-		<xacro:sick_s300_gazebo link="back_laser_link" robot_namespace="${robot_namespace_slashed}" topic="b_scan" />
+		<xacro:sick_s300_gazebo link="front_laser_link" robot_namespace="${robot_namespace_slashed}" topic="f_scan" tf_prefix="${tf_prefix}" />
+		<xacro:sick_s300_gazebo link="back_laser_link" robot_namespace="${robot_namespace_slashed}" topic="b_scan" tf_prefix="${tf_prefix}" />
 		<!-- Settings for the camera of the robot to work in the simulation environment-->
     	<xacro:gazebo_d435 camera_name="${robot_namespace_underscored}camera" reference_link="camera_link" topics_ns="${robot_namespace_slashed}camera" depth_optical_frame="${tf_prefix_slashed}camera_depth_optical_frame" color_optical_frame="${tf_prefix_slashed}camera_color_optical_frame" infrared1_optical_frame="${tf_prefix_slashed}camera_left_ir_optical_frame" infrared2_optical_frame="${tf_prefix_slashed}camera_right_ir_optical_frame" publish_pointcloud="true"/>

File: mir/mir_description/urdf/mir_200/mir_200.gazebo.xacro (robot description, xacro)
@@ -44,6 +44,6 @@
 		<!-- Add Gazebo xacro for the laser scanner to work in Gazebo -->
 		<!-- Please match there macro calls with the sick_s300 xacro calls in the mir_200.urdf.xacro file-->
-		<xacro:sick_s300_gazebo link="front_laser_link" robot_namespace="${robot_namespace_slashed}" topic="f_scan" />
-		<xacro:sick_s300_gazebo link="back_laser_link" robot_namespace="${robot_namespace_slashed}" topic="b_scan" />
+		<xacro:sick_s300_gazebo link="front_laser_link" robot_namespace="${robot_namespace_slashed}" topic="f_scan" tf_prefix="${tf_prefix}" />
+		<xacro:sick_s300_gazebo link="back_laser_link" robot_namespace="${robot_namespace_slashed}" topic="b_scan" tf_prefix="${tf_prefix}" />
 		<!-- Settings for the camera of the robot to work in the simulation environment-->
     	<xacro:gazebo_d435 camera_name="${robot_namespace_underscored}camera" reference_link="camera_link" topics_ns="${robot_namespace_slashed}camera" depth_optical_frame="${tf_prefix_slashed}camera_depth_optical_frame" color_optical_frame="${tf_prefix_slashed}camera_color_optical_frame" infrared1_optical_frame="${tf_prefix_slashed}camera_left_ir_optical_frame" infrared2_optical_frame="${tf_prefix_slashed}camera_right_ir_optical_frame" publish_pointcloud="true"/>
